File: hardware/kicad/MaxPilot.kicad_pcb (KiCad board)
At the start: 2 copper layers, 99.1 x 38.1 mm, 16 parts, among them J1 Conn_01x03, U1 WeMos_D1_mini, U2 MOC3041M, U3 MOC3041M

Commit message: Add L/N/P silkscreen labels on J1 terminal block
Other:
- board text added: "L"
- board text added: "N"
- board text added: "P"
Changed lines of the file:
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@@
+		)
+	)
+	(gr_text "L"
+		(at 12.7 25.4 270)
+		(layer "F.SilkS")
+		(effects
+			(font
+				(size 1 1)
+				(thickness 0.15)
+			)
+			(justify left bottom)
 		)
 	)
@@
 		)
 	)
+	(gr_text "P"
+		(at 12.7 40.64 270)
+		(layer "F.SilkS")
+		(effects
+			(font
+				(size 1 1)
+				(thickness 0.15)
+			)
+			(justify left bottom)
+		)
+	)
+	(gr_text "N"
+		(at 12.7 33.02 270)
+		(layer "F.SilkS")
+		(effects
+			(font
+				(size 1 1)
+				(thickness 0.15)
+			)
+			(justify left bottom)
+		)
+	)
